Commit message: edit urdf

File: whill_description/urdf/whill_model_cr2.urdf (robot description, URDF)
Before this commit: robot whill_model_cr2, 12 links, 11 joints
Joints:
- joint left_front_wheel_joint: axis 0 0 -1 -> 0 0 1; origin xyz=0.330 -0.235 0 rpy=-1.571 0 0 -> xyz=0.330 -0.235 0 rpy=1.57 0 0; type continuous -> fixed
- joint left_wheel_joint: origin xyz=-0.3 0.260 0.015 rpy=1.571 0 0 -> xyz=-0.3 0.260 0.015 rpy=-1.571 0 0
- joint right_front_wheel_joint: axis 0 0 1 -> 0 0 -1; type continuous -> fixed
- joint right_wheel_joint: axis 0 0 -1 -> 0 0 1; origin xyz=-0.3 -0.260 0.015 rpy=-1.571 0 0 -> xyz=-0.3 -0.260 0.015 rpy=1.57 0 0

Commit message: update whill urdf

File: whill_description/urdf/whill_model_cr2.urdf (robot description, URDF)
Before this commit: robot whill_model_cr2, 12 links, 11 joints
Joints:
- joint left_front_wheel_joint: axis 0 0 1 -> 0 0 -1; origin xyz=0.330 -0.235 0 rpy=1.57 0 0 -> xyz=0.330 -0.235 0 rpy=-1.571 0 0
- joint left_wheel_joint: origin xyz=-0.3 0.260 0.015 rpy=-1.571 0 0 -> xyz=-0.3 0.260 0.015 rpy=1.571 0 0
- joint right_front_wheel_joint: axis 0 0 -1 -> 0 0 1
- joint right_wheel_joint: axis 0 0 1 -> 0 0 -1; origin xyz=-0.3 -0.260 0.015 rpy=1.57 0 0 -> xyz=-0.3 -0.260 0.015 rpy=-1.571 0 0
